Commit message: feat(description): positronic_description package with the arm URDF and meshes (#74)
Co-authored-by: Felipe Suassuna <felpssuassuna@gmail.com>
Co-authored-by: Rui Moura <rui2103moura@gmail.com>

File: src/positronic_description/urdf/mycobot_280_jn_sim/mycobot_280_jn_gripper_no_base.urdf (robot description, URDF)
Before this commit: robot mycobot_280_jn, 15 links, 14 joints
Links:
- link gripper_base: mass 0.07075 -> 0.07782; geometry collision mesh filename=package://positronic_description/urdf/mycobot_280_jn_sim/me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; visual mesh filename=package://positronic_description/urdf/mycobot_280_jn_sim/me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
- link gripper_left1: mass 0.00818 -> 0.00900; geometry collision mesh filename=package://positronic_description/urdf/mycobot_280_jn_sim/me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; visual mesh filename=package://positronic_description/urdf/mycobot_280_jn_sim/me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
- link gripper_left2: mass 0.00382 -> 0.00420; geometry collision mesh filename=package://positronic_description/urdf/mycobot_280_jn_sim/me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; visual mesh filename=package://positronic_description/urdf/mycobot_280_jn_sim/me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
- link gripper_left3: mass 0.00262 -> 0.00288; geometry collision mesh filename=package://positronic_description/urdf/mycobot_280_jn_sim/me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; visual mesh filename=package://positronic_description/urdf/mycobot_280_jn_sim/me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
- link gripper_right1: mass 0.00818 -> 0.00900; geometry collision mesh filename=package://positronic_description/urdf/mycobot_280_jn_sim/me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; visual mesh filename=package://positronic_description/urdf/mycobot_280_jn_sim/me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
- link gripper_right2: mass 0.00382 -> 0.00420; geometry collision mesh filename=package://positronic_description/urdf/mycobot_280_jn_sim/me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; visual mesh filename=package://positronic_description/urdf/mycobot_280_jn_sim/me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
- link gripper_right3: mass 0.00262 -> 0.00288; geometry collision mesh filename=package://positronic_description/urdf/mycobot_280_jn_sim/me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; visual mesh filename=package://positronic_description/urdf/mycobot_280_jn_sim/me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
- link joint1: mass 0.51726 -> 0.50875; geometry collision mesh filename=package://positronic_description/urdf/mycobot_280_jn_sim/me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; visual mesh filename=package://positronic_description/urdf/mycobot_280_jn_sim/me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
- link joint2: mass 0.06483 -> 0.06376; geometry collision mesh filename=package://positronic_description/urdf/mycobot_280_jn_sim/me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; visual mesh filename=package://positronic_description/urdf/mycobot_280_jn_sim/me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
- link joint3: mass 0.11472 -> 0.11283; geometry collision mesh filename=package://positronic_description/urdf/mycobot_280_jn_sim/me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; visual mesh filename=package://positronic_description/urdf/mycobot_280_jn_sim/me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
- link joint4: mass 0.09148 -> 0.08998; geometry collision mesh filename=package://positronic_description/urdf/mycobot_280_jn_sim/me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; visual mesh filename=package://positronic_description/urdf/mycobot_280_jn_sim/me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
- link joint5: mass 0.02935 -> 0.02887; geometry collision mesh filename=package://positronic_description/urdf/mycobot_280_jn_sim/me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; visual mesh filename=package://positronic_description/urdf/mycobot_280_jn_sim/me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
- link joint6: mass 0.03671 -> 0.03611; geometry collision mesh filename=package://positronic_description/urdf/mycobot_280_jn_sim/me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; visual mesh filename=package://positronic_description/urdf/mycobot_280_jn_sim/me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
- link joint6_flange: mass 0.00565 -> 0.00556; geometry collision mesh filename=package://positronic_description/urdf/mycobot_280_jn_sim/me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; visual mesh filename=package://positronic_description/urdf/mycobot_280_jn_sim/me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
Joints:
- joint gripper_base_to_gripper_right3: limit lower=-0.15 upper=0.7 effort=10.0 velocity=1.0 -> lower=-0.15 upper=0.8 effort=10.0 velocity=1.0
- joint gripper_left3_to_gripper_left1: limit lower=-0.5 upper=0.5 effort=10.0 velocity=1.0 -> lower=-0.5 upper=0.8 effort=10.0 velocity=1.0
- joint gripper_right3_to_gripper_right1: limit lower=-0.5 upper=0.5 effort=10.0 velocity=1.0 -> lower=-0.8 upper=0.5 effort=10.0 velocity=1.0
- joint joint2_to_joint1: limit lower=-2.9321 upper=2.9321 effort=10.0 velocity=1.0 -> lower=-2.9321 upper=2.9321 effort=10.0 velocity=2.618
- joint joint3_to_joint2: limit lower=-2.4434 upper=2.4434 effort=10.0 velocity=1.0 -> lower=-2.4434 upper=2.4434 effort=10.0 velocity=2.618
- joint joint4_to_joint3: limit lower=-2.6179 upper=2.6179 effort=10.0 velocity=1.0 -> lower=-2.6179 upper=2.6179 effort=10.0 velocity=2.618
- joint joint5_to_joint4: limit lower=-2.6179 upper=2.6179 effort=10.0 velocity=1.0 -> lower=-2.6179 upper=2.6179 effort=10.0 velocity=2.618
- joint joint6_to_joint5: limit lower=-2.7052 upper=2.7925 effort=10.0 velocity=1.0 -> lower=-2.7052 upper=2.7925 effort=10.0 velocity=2.618
- joint joint6output_to_joint6: limit lower=-3.14159 upper=3.14159 effort=10.0 velocity=1.0 -> lower=-3.14159 upper=3.14159 effort=10.0 velocity=2.618

File: src/positronic_description/urdf/mycobot_280_jn_sim/mycobot_280_jn_no_base.urdf (robot description, URDF)
Before this commit: robot mycobot_280_jn, 8 links, 7 joints
Links:
- link joint1: mass 0.51726 -> 0.50875; geometry collision mesh filename=package://positronic_description/urdf/mycobot_280_jn_sim/me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; visual mesh filename=package://positronic_description/urdf/mycobot_280_jn_sim/me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
- link joint2: mass 0.06483 -> 0.06376; geometry collision mesh filename=package://positronic_description/urdf/mycobot_280_jn_sim/me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; visual mesh filename=package://positronic_description/urdf/mycobot_280_jn_sim/me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
- link joint3: mass 0.11472 -> 0.11283; geometry collision mesh filename=package://positronic_description/urdf/mycobot_280_jn_sim/me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; visual mesh filename=package://positronic_description/urdf/mycobot_280_jn_sim/me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
- link joint4: mass 0.09148 -> 0.08998; geometry collision mesh filename=package://positronic_description/urdf/mycobot_280_jn_sim/me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; visual mesh filename=package://positronic_description/urdf/mycobot_280_jn_sim/me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
- link joint5: mass 0.02935 -> 0.02887; geometry collision mesh filename=package://positronic_description/urdf/mycobot_280_jn_sim/me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; visual mesh filename=package://positronic_description/urdf/mycobot_280_jn_sim/me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
- link joint6: mass 0.03671 -> 0.03611; geometry collision mesh filename=package://positronic_description/urdf/mycobot_280_jn_sim/me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; visual mesh filename=package://positronic_description/urdf/mycobot_280_jn_sim/me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
- link joint6_flange: mass 0.00565 -> 0.00556; geometry collision mesh filename=package://positronic_description/urdf/mycobot_280_jn_sim/me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; visual mesh filename=package://positronic_description/urdf/mycobot_280_jn_sim/me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
Joints:
- joint joint2_to_joint1: limit lower=-2.9321 upper=2.9321 effort=10.0 velocity=1.0 -> lower=-2.9321 upper=2.9321 effort=10.0 velocity=2.618
- joint joint3_to_joint2: limit lower=-2.4434 upper=2.4434 effort=10.0 velocity=1.0 -> lower=-2.4434 upper=2.4434 effort=10.0 velocity=2.618
- joint joint4_to_joint3: limit lower=-2.6179 upper=2.6179 effort=10.0 velocity=1.0 -> lower=-2.6179 upper=2.6179 effort=10.0 velocity=2.618
- joint joint5_to_joint4: limit lower=-2.6179 upper=2.6179 effort=10.0 velocity=1.0 -> lower=-2.6179 upper=2.6179 effort=10.0 velocity=2.618
- joint joint6_to_joint5: limit lower=-2.7052 upper=2.7925 effort=10.0 velocity=1.0 -> lower=-2.7052 upper=2.7925 effort=10.0 velocity=2.618
- joint joint6output_to_joint6: limit lower=-3.14159 upper=3.14159 effort=10.0 velocity=1.0 -> lower=-3.14159 upper=3.14159 effort=10.0 velocity=2.618
