Commit message: feat(description): gripper and camera module mounted as on the real arm
joint6output_to_gripper_base turned 180 deg on the flange and the camera
module at 90 deg from the finger line, as seen on the arm on 2026-10-28; the
sign is to be confirmed with the gripper mounted. A roll on camera_link puts
the fingers at the bottom of the image. With this the wrist camera sees both
finger pads and the object between them. Evidence of a pick run in
docs/03_verification/gazebo_pick/docs/figures.

File: src/positronic_description/urdf/mycobot_280_jn_sim/mycobot_280_jn_gripper_camera.urdf (robot description, URDF)
Before this commit: robot mycobot_280_jn, 18 links, 17 joints
Joints:
- joint camera_flange_to_camera_link: origin xyz=0.0415 0.0083 0.0000 rpy=0 0 1.5708 -> xyz=0.0415 0.0083 0.0000 rpy=1.5708 0 1.5708
- joint joint6output_to_camera_flange: origin xyz=0 0 0.01 rpy=1.5708 0 0 -> xyz=0 0 0.01 rpy=1.5708 0 -1.5708
- joint joint6output_to_gripper_base: origin xyz=0 0 0.0505 rpy=1.5708 0 0 -> xyz=0 0 0.0505 rpy=1.5708 0 3.1416
