Commit message: feat(moveit_config):add planning scene for gazebo and rviz

File: src/positronic_description/urdf/positronic_gazebo.urdf.xacro (robot description, xacro)
@@ -9,5 +9,5 @@
   <xacro:arg name="controllers_file" default=""/>
   <!-- Links, joints and meshes of the arm. -->
-  <xacro:include filename="$(find positronic_description)/urdf/mycobot_280_jn_sim/mycobot_280_jn.urdf"/>
+  <xacro:include filename="$(find positronic_description)/urdf/mycobot_280_jn_sim/mycobot_280_jn_gripper_camera.urdf"/>
   <!-- One joint as seen by ros2_control: we command position, we read position. -->
   <xacro:macro name="arm_joint" params="name">
@@ -28,4 +28,9 @@
     <xacro:arm_joint name="joint6_to_joint5"/>
     <xacro:arm_joint name="joint6output_to_joint6"/>
+    <joint name="gripper_controller">
+      <command_interface name="position"/>
+      <state_interface name="position"/>
+      <state_interface name="velocity"/>
+    </joint>
   </ros2_control>
   <!-- Gazebo loads this plugin with the model. It starts the controller_manager with this yaml. -->

Commit message: fix(description): list the gripper finger joints for ros2_control in the Gazebo xacro
The five mimic joints of the adaptive gripper were not in the <ros2_control>
block, so gz_ros2_control never drove them and only one finger link moved.
Listed with a position state interface and no command interface, ros2_control
reads their URDF mimic tags and the Gazebo plugin follows gripper_controller.
A pytest checks the expanded xacro.

File: src/positronic_description/urdf/positronic_gazebo.urdf.xacro (robot description, xacro)
@@ -14,4 +14,13 @@
     <joint name="${name}">
       <command_interface name="position"/>
+      <state_interface name="position"/>
+    </joint>
+  </xacro:macro>
+  <!-- One finger joint as seen by ros2_control: state only. The URDF gives it a mimic tag on
+       gripper_controller, and ros2_control only registers that tag for joints listed here.
+       Registered, gz_ros2_control drives the finger; left out, the Gazebo physics engine
+       ignores the mimic tag and the finger hangs loose. -->
+  <xacro:macro name="finger_joint" params="name">
+    <joint name="${name}">
       <state_interface name="position"/>
     </joint>
@@ -33,4 +42,9 @@
       <state_interface name="velocity"/>
     </joint>
+    <xacro:finger_joint name="gripper_base_to_gripper_left2"/>
+    <xacro:finger_joint name="gripper_left3_to_gripper_left1"/>
+    <xacro:finger_joint name="gripper_base_to_gripper_right3"/>
+    <xacro:finger_joint name="gripper_base_to_gripper_right2"/>
+    <xacro:finger_joint name="gripper_right3_to_gripper_right1"/>
   </ros2_control>
   <!-- Gazebo loads this plugin with the model. It starts the controller_manager with this yaml. -->
